Commit message: chore: remove aip_x1 and rename aip_x1_1 to aip_x1
Signed-off-by: 1222-takeshi <m.takeshi1995@gmail.com>

File: aip_x1_description/urdf/sensor_kit.xacro (robot description, xacro)
@@ -5,5 +5,5 @@
     <xacro:include filename="$(find imu_description)/urdf/imu.xacro"/>
     <xacro:arg name="gpu" default="false"/>
-    <xacro:arg name="config_dir" default="$(find aip_x1_description)/config"/>
+    <xacro:arg name="config_dir" default="$(find aip_x1_1_description)/config"/>
     <xacro:property name="sensor_kit_base_link" default="sensor_kit_base_link"/>
     <joint name="${sensor_kit_base_link}_joint" type="fixed">
@@ -16,5 +16,5 @@
     </link>
     <!-- sensor -->
-    <xacro:property name="calibration" value="${xacro.load_yaml('$(arg config_dir)/sensor_kit_calibration.yaml')}"/>
+    <xacro:property name="calibration" value="${load_yaml('$(arg config_dir)/sensor_kit_calibration.yaml')}"/>
     <!-- lidar -->
     <xacro:PandarXT-32

File: aip_x1_description/urdf/sensors.xacro (robot description, xacro)
@@ -1,7 +1,7 @@
 <?xml version="1.0"?>
 <robot name="vehicle" xmlns:xacro="http://ros.org/wiki/xacro">
-  <xacro:arg name="config_dir" default="$(find aip_x1_description)/config"/>
-  <xacro:include filename="$(find aip_x1_description)/urdf/sensor_kit.xacro"/>
-  <xacro:property name="calibration" value="${xacro.load_yaml('$(arg config_dir)/sensors_calibration.yaml')}"/>
+  <xacro:arg name="config_dir" default="$(find aip_x1_1_description)/config"/>
+  <xacro:include filename="$(find aip_x1_1_description)/urdf/sensor_kit.xacro"/>
+  <xacro:property name="calibration" value="${load_yaml('$(arg config_dir)/sensors_calibration.yaml')}"/>
   <!-- sensor kit -->
   <xacro:sensor_kit_macro

Commit message: chore: remove unused file and fix bug
Signed-off-by: 1222-takeshi <m.takeshi1995@gmail.com>

File: aip_x1_description/urdf/sensor_kit.xacro (robot description, xacro)
@@ -16,5 +16,5 @@
     </link>
     <!-- sensor -->
-    <xacro:property name="calibration" value="${load_yaml('$(arg config_dir)/sensor_kit_calibration.yaml')}"/>
+    <xacro:property name="calibration" value="${xacro.load_yaml('$(arg config_dir)/sensor_kit_calibration.yaml')}"/>
     <!-- lidar -->
     <xacro:PandarXT-32

File: aip_x1_description/urdf/sensors.xacro (robot description, xacro)
@@ -3,5 +3,5 @@
   <xacro:arg name="config_dir" default="$(find aip_x1_description)/config"/>
   <xacro:include filename="$(find aip_x1_description)/urdf/sensor_kit.xacro"/>
-  <xacro:property name="calibration" value="${load_yaml('$(arg config_dir)/sensors_calibration.yaml')}"/>
+  <xacro:property name="calibration" value="${xacro.load_yaml('$(arg config_dir)/sensors_calibration.yaml')}"/>
   <!-- sensor kit -->
   <xacro:sensor_kit_macro

Commit message: replace vlp16 to xt32
Signed-off-by: Autumn60 <harada.akiro@gmail.com>

File: aip_x1_description/urdf/sensor_kit.xacro (robot description, xacro)
@@ -2,38 +2,31 @@
 <robot xmlns:xacro="http://ros.org/wiki/xacro">
   <xacro:macro name="sensor_kit_macro" params="parent x y z roll pitch yaw">
-    <xacro:include filename="$(find velodyne_description)/urdf/VLP-16.urdf.xacro"/>
-    <xacro:include filename="$(find imu_description)/urdf/imu.xacro"/>
-    <xacro:arg name="gpu" default="false"/>
-    <xacro:arg name="config_dir" default="$(find aip_x1_description)/config"/>
-    <xacro:property name="sensor_kit_base_link" default="sensor_kit_base_link"/>
+    <xacro:include filename="$(find pandar_description)/urdf/pandar_xt32.xacro" />
+    <xacro:include filename="$(find imu_description)/urdf/imu.xacro" />
+    <xacro:arg name="gpu" default="false" />
+    <xacro:arg name="config_dir" default="$(find aip_x1_description)/config" />
+    <xacro:property name="sensor_kit_base_link" default="sensor_kit_base_link" />
     <joint name="${sensor_kit_base_link}_joint" type="fixed">
-      <origin rpy="${roll} ${pitch} ${yaw}" xyz="${x} ${y} ${z}"/>
-      <parent link="${parent}"/>
-      <child link="${sensor_kit_base_link}"/>
+      <origin rpy="${roll} ${pitch} ${yaw}" xyz="${x} ${y} ${z}" />
+      <parent link="${parent}" />
+      <child link="${sensor_kit_base_link}" />
     </joint>
     <link name="${sensor_kit_base_link}">
-      <origin rpy="0 0 0" xyz="0 0 0"/>
+      <origin rpy="0 0 0" xyz="0 0 0" />
     </link>
     <!-- sensor -->
-    <xacro:property name="calibration" value="${xacro.load_yaml('$(arg config_dir)/sensor_kit_calibration.yaml')}"/>
+    <xacro:property name="calibration"
+      value="${xacro.load_yaml('$(arg config_dir)/sensor_kit_calibration.yaml')}" />
     <!-- lidar -->
-    <xacro:VLP-16
+    <xacro:PandarXT-32
+      name="pandar_xt32_top"
       parent="sensor_kit_base_link"
-      name="velodyne_top"
-      topic="/points_raw"
-      hz="10"
-      samples="220"
-      gpu="$(arg gpu)"
-    >
-      <origin
-        xyz="${calibration['sensor_kit_base_link']['velodyne_top_base_link']['x']}
-             ${calibration['sensor_kit_base_link']['velodyne_top_base_link']['y']}
-             ${calibration['sensor_kit_base_link']['velodyne_top_base_link']['z']}"
-        rpy="${calibration['sensor_kit_base_link']['velodyne_top_base_link']['roll']}
-             ${calibration['sensor_kit_base_link']['velodyne_top_base_link']['pitch']}
-            ${calibration['sensor_kit_base_link']['velodyne_top_base_link']['yaw']}"
-      />
-    </xacro:VLP-16>
-    <xacro:include filename="$(find pandar_description)/urdf/pandar_xt32.xacro"/>
+      x="${calibration['sensor_kit_base_link']['pandar_xt32_top_base_link']['x']}"
+      y="${calibration['sensor_kit_base_link']['pandar_xt32_top_base_link']['y']}"
+      z="${calibration['sensor_kit_base_link']['pandar_xt32_top_base_link']['z']}"
+      roll="${calibration['sensor_kit_base_link']['pandar_xt32_top_base_link']['roll']}"
+      pitch="${calibration['sensor_kit_base_link']['pandar_xt32_top_base_link']['pitch']}"
+      yaw="${calibration['sensor_kit_base_link']['pandar_xt32_top_base_link']['yaw']}"
+    />
     <xacro:PandarXT-32
       name="pandar_xt32_front_center"

Commit message: fix: change for x1 bench
Signed-off-by: kimurariku <riku.kimura@tier4.co.jp>

File: aip_x1_description/urdf/sensor_kit.xacro (robot description, xacro)
@@ -2,5 +2,5 @@
 <robot xmlns:xacro="http://ros.org/wiki/xacro">
   <xacro:macro name="sensor_kit_macro" params="parent x y z roll pitch yaw">
-    <xacro:include filename="$(find velodyne_description)/urdf/VLP-16.urdf.xacro"/>
+    <xacro:include filename="$(find pandar_description)/urdf/pandar_xt32.xacro"/>
     <xacro:include filename="$(find imu_description)/urdf/imu.xacro"/>
     <xacro:arg name="gpu" default="false"/>
@@ -18,21 +18,14 @@
     <xacro:property name="calibration" value="${xacro.load_yaml('$(arg config_dir)/sensor_kit_calibration.yaml')}"/>
     <!-- lidar -->
-    <xacro:VLP-16
+    <xacro:PandarXT-32
+      name="pandar_xt32_top"
       parent="sensor_kit_base_link"
-      name="velodyne_top"
-      topic="/points_raw"
-      hz="10"
-      samples="220"
-      gpu="$(arg gpu)"
-    >
-      <origin
-        xyz="${calibration['sensor_kit_base_link']['velodyne_top_base_link']['x']}
-             ${calibration['sensor_kit_base_link']['velodyne_top_base_link']['y']}
-             ${calibration['sensor_kit_base_link']['velodyne_top_base_link']['z']}"
-        rpy="${calibration['sensor_kit_base_link']['velodyne_top_base_link']['roll']}
-             ${calibration['sensor_kit_base_link']['velodyne_top_base_link']['pitch']}
-            ${calibration['sensor_kit_base_link']['velodyne_top_base_link']['yaw']}"
-      />
-    </xacro:VLP-16>
+      x="${calibration['sensor_kit_base_link']['pandar_xt32_top_base_link']['x']}"
+      y="${calibration['sensor_kit_base_link']['pandar_xt32_top_base_link']['y']}"
+      z="${calibration['sensor_kit_base_link']['pandar_xt32_top_base_link']['z']}"
+      roll="${calibration['sensor_kit_base_link']['pandar_xt32_top_base_link']['roll']}"
+      pitch="${calibration['sensor_kit_base_link']['pandar_xt32_top_base_link']['pitch']}"
+      yaw="${calibration['sensor_kit_base_link']['pandar_xt32_top_base_link']['yaw']}"
+    />
     <xacro:include filename="$(find pandar_description)/urdf/pandar_xt32.xacro"/>
     <xacro:PandarXT-32

Commit message: replace vlp-16 to xt-32 in aip_x1_description
Signed-off-by: Autumn60 <harada.akiro@gmail.com>

File: aip_x1_description/urdf/sensor_kit.xacro (robot description, xacro)
@@ -2,5 +2,5 @@
 <robot xmlns:xacro="http://ros.org/wiki/xacro">
   <xacro:macro name="sensor_kit_macro" params="parent x y z roll pitch yaw">
-    <xacro:include filename="$(find velodyne_description)/urdf/VLP-16.urdf.xacro"/>
+    <xacro:include filename="$(find pandar_description)/urdf/pandar_xt32.xacro"/>
     <xacro:include filename="$(find imu_description)/urdf/imu.xacro"/>
     <xacro:arg name="gpu" default="false"/>
@@ -18,22 +18,14 @@
     <xacro:property name="calibration" value="${xacro.load_yaml('$(arg config_dir)/sensor_kit_calibration.yaml')}"/>
     <!-- lidar -->
-    <xacro:VLP-16
+    <xacro:PandarXT-32
+      name="pandar_xt32_top"
       parent="sensor_kit_base_link"
-      name="velodyne_top"
-      topic="/points_raw"
-      hz="10"
-      samples="220"
-      gpu="$(arg gpu)"
-    >
-      <origin
-        xyz="${calibration['sensor_kit_base_link']['velodyne_top_base_link']['x']}
-             ${calibration['sensor_kit_base_link']['velodyne_top_base_link']['y']}
-             ${calibration['sensor_kit_base_link']['velodyne_top_base_link']['z']}"
-        rpy="${calibration['sensor_kit_base_link']['velodyne_top_base_link']['roll']}
-             ${calibration['sensor_kit_base_link']['velodyne_top_base_link']['pitch']}
-            ${calibration['sensor_kit_base_link']['velodyne_top_base_link']['yaw']}"
-      />
-    </xacro:VLP-16>
-    <xacro:include filename="$(find pandar_description)/urdf/pandar_xt32.xacro"/>
+      x="${calibration['sensor_kit_base_link']['pandar_xt32_top_base_link']['x']}"
+      y="${calibration['sensor_kit_base_link']['pandar_xt32_top_base_link']['y']}"
+      z="${calibration['sensor_kit_base_link']['pandar_xt32_top_base_link']['z']}"
+      roll="${calibration['sensor_kit_base_link']['pandar_xt32_top_base_link']['roll']}"
+      pitch="${calibration['sensor_kit_base_link']['pandar_xt32_top_base_link']['pitch']}"
+      yaw="${calibration['sensor_kit_base_link']['pandar_xt32_top_base_link']['yaw']}"
+    />
     <xacro:PandarXT-32
       name="pandar_xt32_front_center"
